File: StarLEDBoard.kicad_sch (KiCad schematic)
At the start: 9 parts, among them J1 Conn_01x02_Socket

Commit message: Ordered Board
Parts:
- J1: footprint (none) -> Library:LEDConnector
Other:
- moved on the sheet: D1, D2, D3, D4
Changed lines of the file:
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@@
 	(paper "A4")
 	(label "LED+"
-		(at 161.29 96.52 90)
+		(at 166.37 96.52 90)
 		(effects
 			(font
@@
 	)
 	(label "LED-"
-		(at 161.29 127 270)
+		(at 166.37 127 270)
 		(effects
 			(font
@@
 	(symbol
 		(lib_id "Device:LED")
-		(at 161.29 107.95 90)
+		(at 166.37 107.95 90)
 		(unit 1)
 		(exclude_from_sim no)
@@
 		(fields_autoplaced yes)
 		(property "Reference" "D3"
-			(at 159.258 110.7497 90)
+			(at 164.338 110.7497 90)
 			(effects
 				(font
@@
 		)
 		(property "Value" "LED"
-			(at 159.258 108.3254 90)
+			(at 164.338 108.3254 90)
 			(effects
 				(font
@@
 		)
 		(property "Footprint" "LED_SMD:LED_Everlight-SMD3528_3.5x2.8mm_67-21ST"
-			(at 161.29 107.95 0)
-			(effects
-				(font
-					(size 1.27 1.27)
-				)
-				(hide yes)
-			)
-		)
-		(property "Datasheet" "~"
-			(at 161.29 107.95 0)
+			(at 166.37 107.95 0)
+			(effects
+				(font
+					(size 1.27 1.27)
+				)
+				(hide yes)
+			)
+		)
+		(property "Datasheet" "~"
+			(at 166.37 107.95 0)
 			(effects
 				(font
@@
 		)
 		(property "Description" "Light emitting diode"
-			(at 161.29 107.95 0)
+			(at 166.37 107.95 0)
 			(effects
 				(font
@@
 		)
 		(property "Sim.Pins" "1=K 2=A"
-			(at 161.29 107.95 0)
+			(at 166.37 107.95 0)
 			(effects
 				(font
@@
 	(symbol
 		(lib_id "Device:LED")
-		(at 161.29 100.33 90)
+		(at 166.37 100.33 90)
 		(unit 1)
 		(exclude_from_sim no)
@@
 		(fields_autoplaced yes)
 		(property "Reference" "D4"
-			(at 159.258 103.1297 90)
+			(at 164.338 103.1297 90)
 			(effects
 				(font
@@
 		)
 		(property "Value" "LED"
-			(at 159.258 100.7054 90)
+			(at 164.338 100.7054 90)
 			(effects
 				(font
@@
 		)
 		(property "Footprint" "LED_SMD:LED_Everlight-SMD3528_3.5x2.8mm_67-21ST"
-			(at 161.29 100.33 0)
-			(effects
-				(font
-					(size 1.27 1.27)
-				)
-				(hide yes)
-			)
-		)
-		(property "Datasheet" "~"
-			(at 161.29 100.33 0)
+			(at 166.37 100.33 0)
+			(effects
+				(font
+					(size 1.27 1.27)
+				)
+				(hide yes)
+			)
+		)
+		(property "Datasheet" "~"
+			(at 166.37 100.33 0)
 			(effects
 				(font
@@
 		)
 		(property "Description" "Light emitting diode"
-			(at 161.29 100.33 0)
+			(at 166.37 100.33 0)
 			(effects
 				(font
@@
 		)
 		(property "Sim.Pins" "1=K 2=A"
-			(at 161.29 100.33 0)
+			(at 166.37 100.33 0)
 			(effects
 				(font
@@
 	(symbol
 		(lib_id "Device:LED")
-		(at 161.29 115.57 90)
+		(at 166.37 115.57 90)
 		(unit 1)
 		(exclude_from_sim no)
@@
 		(fields_autoplaced yes)
 		(property "Reference" "D2"
-			(at 159.258 118.3697 90)
+			(at 164.338 118.3697 90)
 			(effects
 				(font
@@
 		)
 		(property "Value" "LED"
-			(at 159.258 115.9454 90)
+			(at 164.338 115.9454 90)
 			(effects
 				(font
@@
 		)
 		(property "Footprint" "LED_SMD:LED_Everlight-SMD3528_3.5x2.8mm_67-21ST"
-			(at 161.29 115.57 0)
-			(effects
-				(font
-					(size 1.27 1.27)
-				)
-				(hide yes)
-			)
-		)
-		(property "Datasheet" "~"
-			(at 161.29 115.57 0)
+			(at 166.37 115.57 0)
+			(effects
+				(font
+					(size 1.27 1.27)
+				)
+				(hide yes)
+			)
+		)
+		(property "Datasheet" "~"
+			(at 166.37 115.57 0)
 			(effects
 				(font
@@
 		)
 		(property "Description" "Light emitting diode"
-			(at 161.29 115.57 0)
+			(at 166.37 115.57 0)
 			(effects
 				(font
@@
 		)
 		(property "Sim.Pins" "1=K 2=A"
-			(at 161.29 115.57 0)
+			(at 166.37 115.57 0)
 			(effects
 				(font
@@
 			)
 		)
-		(property "Footprint" ""
+		(property "Footprint" "Library:LEDConnector"
 			(at 186.69 109.22 0)
 			(effects
@@
 	(symbol
 		(lib_id "Device:LED")
-		(at 161.29 123.19 90)
+		(at 166.37 123.19 90)
 		(unit 1)
 		(exclude_from_sim no)
@@
 		(fields_autoplaced yes)
 		(property "Reference" "D1"
-			(at 159.258 125.9897 90)
+			(at 164.338 125.9897 90)
 			(effects
 				(font
@@
 		)
 		(property "Value" "LED"
-			(at 159.258 123.5654 90)
+			(at 164.338 123.5654 90)
 			(effects
 				(font
@@
 		)
 		(property "Footprint" "LED_SMD:LED_Everlight-SMD3528_3.5x2.8mm_67-21ST"
-			(at 161.29 123.19 0)
-			(effects
-				(font
-					(size 1.27 1.27)
-				)
-				(hide yes)
-			)
-		)
-		(property "Datasheet" "~"
-			(at 161.29 123.19 0)
+			(at 166.37 123.19 0)
+			(effects
+				(font
+					(size 1.27 1.27)
+				)
+				(hide yes)
+			)
+		)
+		(property "Datasheet" "~"
+			(at 166.37 123.19 0)
 			(effects
 				(font
@@
 		)
 		(property "Description" "Light emitting diode"
-			(at 161.29 123.19 0)
+			(at 166.37 123.19 0)
 			(effects
 				(font
@@
 		)
 		(property "Sim.Pins" "1=K 2=A"
-			(at 161.29 123.19 0)
-			(effects
-				(font
+			(at 166.37 123.19 0)
+			(effects
+				(font
